File: Esquemático: nRF52832/Esquemático: nRF52832.sch (KiCad schematic (older format))
At the start: 18 parts, among them X1 32MHz, X2 32.768kHz

Commit message: Add files via upload
Parts:
- C1, C11, C12, C2: value 12pF -> 12p
- C10: value 1.0µF -> 1.0µ
- C3: value 0.8pF -> 0.8p
- C4, C8: value 100nF -> 100n
- C5: renamed from C3; value C -> 100n
- C7: value 100pF -> 100p
- C9: value 4.7µF -> 4.7µ
- L2: value 10µH -> 10µ
- L3: value 15nH -> 15n
- gave numbers to parts that had none: 1
Connections:
- net at L1.1, U1.30 (ANT): now also C3.1
- net at L3.1, U1.46 (DEC4): now also C10.1
- no-connect marks 0 -> 33
Other:
- moved on the sheet: C1, C10, C11, C12, C2, C3, C4, C5, C6, C7, C8, C9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
