File: Esquemático: nRF52832/Esquem__tico_ nRF52832.kicad_pcb (KiCad board)
At the start: 2 copper layers, 27.9 x 20.3 mm, 18 parts, among them U1 nRF52832, X1 32MHz, X2 32.768kHz

Commit message: Add files via upload
Parts:
- moved C4 0.20 mm to (178.3, 86.4)
Routing:
- net Net-(C12-Pad1): track 8.02 -> 8.66 mm
- net Earth: track 32.5 -> 31.9 mm
- net Net-(L2-Pad2): track 1.65 -> 2.19 mm
- net Net-(C11-Pad1): track 5.24 -> 5.78 mm
- net Net-(C3-Pad1): track 4.65 -> 5.16 mm
Other:
- net class Default: clearance 0.2 -> 0
- rule trace_clearance: 0.2 -> 0
